Commit message: updated parameters as per real robot

File: ur_description/urdf/ur10.urdf.xacro (robot description, xacro)
@@ -8,5 +8,5 @@
   <xacro:include filename="$(find ur_description)/urdf/ur.gazebo.xacro" />
   <xacro:property name="pi" value="3.14159265" />
-  <xacro:property name="ee_length" value="0.23" /> <!-- 0.2 is good -->
+  <xacro:property name="ee_length" value="0.23" /> <!-- 0.2 is end effector metal, 0.3 for vacuum on the end -->
   <xacro:property name="ee_radius" value="0.01" /> <!-- 0.01 is good -->
   <!-- Inertia parameters -->

File: ur_description/urdf/ur10_robot.urdf.xacro (robot description, xacro)
@@ -12,5 +12,5 @@
     <parent link="world" />
     <child link = "base_link" />
-    <origin xyz="0.0 0.0 0.0" rpy="0.0 0.0 0.0" />
+    <origin xyz="0.0 0.0 0.963" rpy="0.0 0.0 0.0" />
   </joint>
 </robot>
